Commit message: feat: complete campus autonomous navigation stack, 3D LiDAR/camera safety pipeline, and tooling

File: src/CART_description/urdf/CART.xacro (robot description, xacro)
@@ -15,5 +15,5 @@
       <mesh filename="file://$(find CART_description)/meshes/base_link.stl" scale="0.1 0.1 0.1" />
     </geometry>
-    <material name="silver" />
+    <material name="safety_orange" />
   </visual>
   <collision>
@@ -35,5 +35,5 @@
       <mesh filename="file://$(find CART_description)/meshes/wheel_front_left_1.stl" scale="0.1 0.1 0.1" />
     </geometry>
-    <material name="silver" />
+    <material name="rubber_black" />
   </visual>
   <collision>
@@ -55,5 +55,5 @@
       <mesh filename="file://$(find CART_description)/meshes/wheel_front_right_1.stl" scale="0.1 0.1 0.1" />
     </geometry>
-    <material name="silver" />
+    <material name="rubber_black" />
   </visual>
   <collision>
@@ -75,5 +75,5 @@
       <mesh filename="file://$(find CART_description)/meshes/top_1.stl" scale="0.1 0.1 0.1" />
     </geometry>
-    <material name="silver" />
+    <material name="canopy_white" />
   </visual>
   <collision>
@@ -95,5 +95,5 @@
       <mesh filename="file://$(find CART_description)/meshes/wheel_back_left_1.stl" scale="0.1 0.1 0.1" />
     </geometry>
-    <material name="silver" />
+    <material name="rubber_black" />
   </visual>
   <collision>
@@ -115,5 +115,5 @@
       <mesh filename="file://$(find CART_description)/meshes/wheel_back_right_1.stl" scale="0.1 0.1 0.1" />
     </geometry>
-    <material name="silver" />
+    <material name="rubber_black" />
   </visual>
   <collision>
@@ -135,5 +135,5 @@
       <mesh filename="file://$(find CART_description)/meshes/Knuckle_left_1.stl" scale="0.1 0.1 0.1" />
     </geometry>
-    <material name="silver" />
+    <material name="rubber_black" />
   </visual>
   <collision>
@@ -155,5 +155,5 @@
       <mesh filename="file://$(find CART_description)/meshes/knuckle_right_1.stl" scale="0.1 0.1 0.1" />
     </geometry>
-    <material name="silver" />
+    <material name="rubber_black" />
   </visual>
   <collision>
@@ -207,3 +207,24 @@
   <limit upper="0.523599" lower="-0.523599" effort="100" velocity="100" />
 </joint>
-<gazebo><plugin filename="gz-sim-ackermann-steering-system" name="gz::sim::systems::AckermannSteering"><left_joint>Revolute 20</left_joint><right_joint>Revolute 21</right_joint><left_steering_joint>Revolute 22</left_steering_joint><right_steering_joint>Revolute 23</right_steering_joint><kingpin_width>0.755</kingpin_width><steering_limit>0.8</steering_limit><wheel_base>2.124</wheel_base><wheel_radius>0.277</wheel_radius><min_velocity>-5</min_velocity><max_velocity>5</max_velocity><topic>/cmd_vel</topic></plugin></gazebo></robot>
+<gazebo>
+  <plugin filename="gz-sim-ackermann-steering-system" name="gz::sim::systems::AckermannSteering">
+    <left_joint>Revolute 20</left_joint>
+    <right_joint>Revolute 21</right_joint>
+    <left_steering_joint>Revolute 22</left_steering_joint>
+    <right_steering_joint>Revolute 23</right_steering_joint>
+    <kingpin_width>0.755</kingpin_width>
+    <steering_limit>0.8</steering_limit>
+    <wheel_base>2.124</wheel_base>
+    <wheel_radius>0.277</wheel_radius>
+    <min_velocity>-5</min_velocity>
+    <max_velocity>5</max_velocity>
+    <topic>/cmd_vel</topic>
+  </plugin>
+  <plugin filename="gz-sim-odometry-publisher-system" name="gz::sim::systems::OdometryPublisher">
+    <odom_frame>world</odom_frame>
+    <robot_base_frame>base_link</robot_base_frame>
+    <odom_topic>/model/CART/odometry_world</odom_topic>
+    <dimensions>3</dimensions>
+  </plugin>
+</gazebo>
+</robot>

File: src/CART_description/urdf/materials.xacro (robot description, xacro)
@@ -4,3 +4,12 @@
   <color rgba="0.700 0.700 0.700 1.000"/>
 </material>
+<material name="safety_orange">
+  <color rgba="1.000 0.350 0.000 1.000"/>
+</material>
+<material name="canopy_white">
+  <color rgba="0.950 0.950 0.950 1.000"/>
+</material>
+<material name="rubber_black">
+  <color rgba="0.100 0.100 0.100 1.000"/>
+</material>
 </robot>
